File: PlacaMirasso.kicad_pcb (KiCad board)
At the start: 2 copper layers, 78.1 x 78.7 mm, 94 parts, among them J1 USB_OTG, J10 GS2, J11 GS2, J12 GS2, J13 GS2, J14 ANALIZER_ADXL, J15 ANALIZER_MPU, J17 SPI_ANALYZER, J18 BAT, J2 DEBUG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

Commit message: [Bd] First PCB draft
Parts:
- removed J5: GND, Pin_Headers:Pin_Header_Straight_1x02_Pitch2.54mm
- added G***: LOGO, TOROID:Logo_7_06mm_FSilk, F.Cu at (137.8, 101.6)
- J2: footprint Pin_Headers:Pin_Header_Straight_1x02_Pitch2.54mm -> Pin_Headers:Pin_Header_Straight_1x03_Pitch2.54mm
- P1, P2: footprint Pin_Headers:Pin_Header_Straight_1x08_Pitch2.54mm -> Socket_Strips:Socket_Strip_Straight_1x08_Pitch2.54mm
- moved J17 10.2 mm to (157.5, 133.6), turned to 270 degrees
- moved J2 1.14 mm to (154.9, 137.3)
Connections:
- J17 pad 1: /SPI1_CS_1 -> /SPI1_CS_2
- J17 pad 2: /SPI1_SCK -> /SPI1_MOSI
- J17 pad 4: /SPI1_MOSI -> /SPI1_SCK
- J17 pad 5: /SPI1_CS_2 -> /SPI1_CS_1
Routing:
- net /U5V: track 48.5 -> 46.7 mm
- net /VBAT_ADC: track 64.9 -> 63.3 mm
- net /DEBUG_RX_uC: track 16.9 -> 17.9 mm
- net /DEBUG_TX_uC: track 15.0 -> 16.0 mm
- net GND: track 88.7 -> 87.9 mm
- net Net-(C14-Pad1): track 16.4 -> 15.6 mm
- net /I2C1_SCL: track 67.9 -> 67.2 mm
- net /SPI1_CS_1: track 25.9 -> 25.3 mm
Other:
- net class Default: clearance 0.2 -> 0
- rule trace_clearance: 0.2 -> 0
- board text added: "3517 FIng - UNCu fclad@toroid.io"
- board text removed: "fcladera@fcladera.com"

Commit message: [Bd] Second draft
Parts:
- MNT1, MNT2, MNT3, MNT4: footprint Mounting_Holes:MountingHole_3.2mm_M3 -> Mounting_Holes:MountingHole_2.2mm_M2_Pad
- moved MNT2 0.18 mm to (177.7, 76.3)
- moved MNT3 0.18 mm to (177.7, 126.9)
- moved MNT1 0.18 mm to (127.1, 76.3)
- moved MNT4 0.18 mm to (127.1, 126.9)
Routing:
- net /E5V: track 15.1 -> 16.5 mm
- net Net-(C14-Pad1): track 15.6 -> 16.4 mm
Other:
- board text added: "1735 FIng - UNCu fclad@toroid.io"
- board text removed: "3517 FIng - UNCu fclad@toroid.io"
